Commit message: Tidy up exercise .urdf

File: urdf/thymio_simple.urdf.xacro (robot description, xacro)
@@ -5,8 +5,4 @@
     <xacro:include filename="$(find ros_basics_models)/urdf/utils/custom_sensors.xacro" />
     <xacro:include filename="$(find ros_basics_exercise)/urdf/thymio_simple.gazebo" />
-    <xacro:arg name="left_wheel_mu" default="100.0"/>
-    <xacro:property name="left_wheel_mu_p" value="$(arg left_wheel_mu)"/>
-    <xacro:arg name="right_wheel_mu" default="100.0"/>
-    <xacro:property name="right_wheel_mu_p" value="$(arg right_wheel_mu)"/>
     <xacro:property name="wheel_radius" value="0.022"/>
     <xacro:property name="wheel_len" value="0.015"/>
@@ -30,4 +26,8 @@
             <material name="white"/>
         </collision>
+        <inertial>
+            <mass value="${body_mass}"/>
+            <xacro:box_inertia mass="${body_mass}" x="0.11" y="0.112" z="0.045" />
+        </inertial>
         <!-- Implement the caster wheel -->
     </link>
